File: d-cube.sch (EAGLE design)
At the start: 63 parts, among them IC1 74AC86D, IC2 SFH6156, IC3 SFH6156, IC4 ISO7220M, IC5 ISO7221M, IC7 NXE2, IC8 ADUM3160, U3 COMPLEMENTARY

Commit message: Update to 2.1
Parts:
- removed IGND: LSP10, solpad:LSP10
- removed J1: (no value), SparkFun-Connectors:M02PTH3
- removed NS1, NS2: SSW-112-02-S-S, con-samtec:SSW-112-02-S-S
- removed Q1, Q2: (no value), transistors:2N7002_SOT23
- removed SV1: (no value), con-lstb:MA13-2
- removed SV2: (no value), con-lstb:MA07-2
- removed U3: COMPLEMENTARY, mos:COMPLEMENTARY
- removed USB_TARGET: PN87520-S, con-berg:PN87520-S
- added C20, C21, C22, C23, C24, C25, C26, C27, C29, C3, C5: 0.1u, SparkFun-Passives:CAP0402-CAP
- added C30: 470u, rcl:CPOL-EUCT7343
- added C31: 1000uF, SparkFun-Capacitors:560UF-PANASONIC_G-25V-20%
- added C32: 0.1u, SparkFun-Passives:CAP0805
- added C33, C34: 0.1uF, SparkFun-Capacitors:0.1UF-0402-16V-10%
- added C35: 10n, SparkFun-Passives:CAP0805
- added C36: 10uF, SparkFun-Capacitors:10UF-0805-10V-10%
- added C37, C38: 1.0uF, SparkFun-Capacitors:1.0UF-0805-25V-10%
- added GPIO: (no value), SparkFun-Connectors:CONN_09NO_SILK
- added GPS_ANT: BU-SMA-V, con-coax:BU-SMA-V
- added I2C: (no value), SparkFun-Connectors:CONN_021X02_NO_SILK
- added IC10, IC11, IC9: SI8640AB-B-IS1, silabslbr:SI8640AB-B-IS1
- added IC12: 24AA32ASM, microchip:24AA32ASM
- added IC13: I2C EEPROM, SparkFun-IC-Memory:EEPROM-I2CEIAJ
- added IC14: NEO-M8, ubloxLib:NEO-M8
- added IC15: MIC550X-YM5, borkedlabs-powerics:MIC550X-YM5
- added IC16: COMPLEMENTARY, mos:COMPLEMENTARY
- added IC17, IC18: 74LVC1G04, SparkFun-DigitalIC:INVERTER_SOT353-5
- added L3: 27nH, SparkFun-Coils:INDUCTOR-0402-3.9NH
- added LAN_IN: SI-52008-F, con-pulse:SI-52008-F
- added LAN_PI: 0446200002, con-molex:0446200002
- added POE: (no value), my-con:CONN_02X2
- added R21, R22, R23, R24, R29, R30, R31, R32: 100, SparkFun-Passives:RESISTOR0402-RES
- added R25, R26, R27, R28, R35: 100k, SparkFun-Passives:RESISTOR0402-RES
- added R33, R34: 10k, SparkFun-Passives:RESISTOR0402-RES
- added R36: 220, SparkFun-Passives:RESISTOR0402-RES
- added R37: 470, SparkFun-Passives:RESISTOR0402-RES
- added R38: 10, SparkFun-Passives:RESISTOR0402-RES
- added R40, R41: 100k, SparkFun-Resistors:RESISTOR0402
- added RPI: (no value), con-lstb:MA20-2
- added SV5: (no value), con-lstb:MA06-1
- added SV6: (no value), con-lstb:MA04-1
- added TP_3V3, TP_IGND, TP_IGND1, TP_VCC: LSP10, solpad:LSP10
- added USB_TGT: PN87520-S, con-berg:PN87520-S
- C1, C2: value 100n -> 0.1u; device SparkFun-Passives:CAP0805 -> SparkFun-Passives:CAP0402-CAP
- C10, C11, C12, C13, C14, C15, C16, C17, C18, C19, C7, C8, C9: device SparkFun-Passives:CAP0805 -> SparkFun-Passives:CAP0402-CAP
- IC1: value 74AC86D -> SI8605; device 74xx-eu:74AC86D -> silabslbr:SI8605
- IC2, IC3: value SFH6156 -> SI8640AB-B-IS1; device optocoupler:SFH6156 -> silabslbr:SI8640AB-B-IS1
- R1: value 3k3 -> 10k; device SparkFun-Passives:RESISTOR0805-RES -> SparkFun-Passives:RESISTOR0402-RES
- R10, R11, R12, R13, R15, R17, R18, R19, R20, R6, R7, R9: device SparkFun-Passives:RESISTOR0805-RES -> SparkFun-Passives:RESISTOR0402-RES
- R2, R3: value 470 -> 100k; device SparkFun-Passives:RESISTOR0805-RES -> SparkFun-Passives:RESISTOR0402-RES
- R4, R5: value 10k -> 100k; device SparkFun-Passives:RESISTOR0805-RES -> SparkFun-Passives:RESISTOR0402-RES
Connections:
- removed net 5V_SW: C4.1, L1.1, U3B.D
- removed net GPIO1: IC1A.I1, IC2CE.C, NS2-5.1, R1.1, R5.1, SV1.12
- removed net GPIO2: IC3CE.C, R4.1, SV1.11
- removed net GPIO3: R20.1, R6.2, SV1.16
- removed net GPIO_EDGE: IC1A.O, NS2-10.1
- removed net GPIO_LP: C1.1, IC1A.I0, R1.2
- removed net GPIO_TARGET: J1.1, Q1.G
- removed net RESET_TARGET: J1.2, Q2.G
- removed net VCCIO: NS2-3.1
- new net !EN_BLOCK1: IC17.Y, IC2.EN
- new net !EN_BLOCK2: IC18.Y, IC3.EN
- new net AIN: IC1.ADIN
- new net AOUT: IC1.ADOUT
- new net B1C1: R21.2, RPI.11
- new net B1C2: R22.2, RPI.7
- new net B1C3: R23.2, RPI.12
- new net B1C4: R24.2, RPI.13
- new net B2C1: R29.2, RPI.15
- new net B2C2: R30.2, RPI.16
- new net B2C3: R31.2, RPI.18
- new net B2C4: R32.2, RPI.22
- new net BIN: IC1.BDIN
- new net BOUT: IC1.BDOUT
- new net BSCL: I2C.1, IC1.BSCL, R41.1
- new net BSDA: I2C.2, IC1.BSDA, R40.1
- new net CP1: R1.2, SV5.5
- new net CP2: R1.1, SV5.6
- new net CT: LAN_IN.CT
- new net EN_BLOCK1: IC11.INB, IC17.A, R34.2, RPI.36
- new net EN_BLOCK2: IC11.INC, IC18.A, R33.2, RPI.32
- new net GPS_SIG: GPS_ANTG$1.1, IC14.11_RF_IN, L3.1
- new net GSCL: IC12.SCL, IC14.19_SCL/SPI_CLK
- new net GSDA: IC12.SDA, IC14.18_SDA/SPI_CS_N
- new net I_B1C1: GPIO.4, R2.2
- new net I_B1C2: GPIO.3, R3.2
- new net I_B1C3: GPIO.2, R4.2
- new net I_B1C4: GPIO.1, R5.2
- new net I_B2C1: GPIO.8, R25.2
- new net I_B2C2: GPIO.7, R26.2
- new net I_B2C3: GPIO.6, R27.2
- new net I_B2C4: GPIO.5, R28.2
- new net I_EN_BLOCK1: IC10.EN, IC11.OUTB
- new net I_EN_BLOCK2: IC11.OUTC, IC9.EN
- new net I_PWR_SW: IC11.OUTA, R20.1, R6.2
- new net I_RST_SW: GPIO.9, IC11.OUTD
- new net N$10: LAN_IN.A-L, R37.2
- new net N$13: IC10.OUTD, IC2.IND, R5.1
- new net N$15: IC10.OUTB, IC2.INB, R3.1
- new net N$21: IC10.IND, IC2.OUTD, R21.1
- new net N$23: IC3.IND, IC9.OUTD, R28.1
- new net N$24: IC3.INC, IC9.OUTC, R27.1
- new net N$25: IC3.INB, IC9.OUTB, R26.1
- new net N$26: IC3.OUTA, IC9.INA, R32.1
- new net N$27: IC3.OUTB, IC9.INB, R31.1
- new net N$28: IC3.OUTC, IC9.INC, R30.1
- new net N$29: IC3.OUTD, IC9.IND, R29.1
- new net N$30: IC14.8_RESET_N, IC14.9_VCC_RF, R38.2
- new net N$32: C35.1, L3.2, R38.1
- new net N$6: IC10.INA, IC2.OUTA, R24.1
- new net N$7: IC10.INB, IC2.OUTB, R23.1
- new net N$9: LAN_IN.A-R, R36.2
- new net OADJ: R35.1, SV6.3
- new net PPS: IC14.3_TIMEPULSE, RPI.37
- new net PWR_SW: IC11.INA, RPI.40
- new net RST_SW: IC11.IND, RPI.38
- new net RX+: LAN_IN.RD+, LAN_PI.3
- new net RX-: LAN_IN.RD-, LAN_PI.6
- new net SCL: IC1.ASCL, IC13.SCL, RPI.5
- new net SDA: IC1.ASDA, IC13.SDA, RPI.3
- new net TX+: LAN_IN.TD+, LAN_PI.1
- new net TX-: LAN_IN.TD-, LAN_PI.2
- new net VCC/2: C2.1, C21.1, C24.1, C3.1, C34.1, C38.1, C5.1, IC1.VCC2, IC10.VCC2, IC11.EN, IC11.VCC2, IC15.VOUT, IC2.VCC1, IC3.VCC1, IC9.VCC2, R40.2, R41.2, TP_3V3.MP
- new net VCC_SW: IC16B.D, TP_VCC.MP, USB_TGT.1, V.1
- new net VINA+: LAN_IN.VC2+, POE.2, SV5.1
- new net VINA-: LAN_IN.VC2-, POE.1, SV5.2
- new net VINB+: LAN_IN.VC1+, POE.4, SV5.3
- new net VINB-: LAN_IN.VC1-, POE.3, SV5.4
- net +3V3: now also C1.1, C20.1, C22.1, C23.1, C25.1, C26.1, C27.1, C29.1, C33.1, C36.1, IC1.VCC1, IC10.VCC1, IC11.VCC1, IC12.VCC, IC13.VCC, IC14.22_V_BCKP, IC14.23_VCC, IC17.VCC, IC18.VCC, IC2.VCC2, IC3.VCC2, IC9.VCC1, R36.1, RPI.1, RPI.17; no longer C2.1, IC1P.VCC, R4.2, R5.2, SV1.1, SV1.17
- net +5V: now also C30.+, C31.+, C32.1, R37.1, RPI.2, RPI.4, SV6.2; no longer NS2-1.1, SV1.2, SV1.4
- net CSB: now also RPI.24; no longer SV1.24
- net D+_OUT_TERM: now also USB_TGT.3; no longer USB_TARGET.3
- net D-_OUT_TERM: now also USB_TGT.2; no longer USB_TARGET.2
- net GND: now also C20.2, C22.2, C23.2, C25.2, C26.2, C27.2, C29.2, C30.-, C31.-, C32.2, C33.2, C35.2, C36.2, GPS_ANTG$1.GND, IC1.GND1, IC10.GND1@1, IC10.GND1@2, IC11.GND1@1, IC11.GND1@2, IC12.A0, IC12.A1, IC12.A2, IC12.GND, IC12.WP, IC13.A0, IC13.A1, IC13.A2, IC13.VSS, IC14.10_GND, IC14.12_GND, IC14.13_GND, IC14.24_GND, IC14.7_VDD_USB, IC17.GND, IC18.GND, IC2.GND2@1, IC2.GND2@2, IC3.GND2@1, IC3.GND2@2, IC9.GND1@1, IC9.GND1@2, LAN_IN.C-L, LAN_IN.C-R, LAN_IN.SHIELD@1, LAN_IN.SHIELD@2, LAN_PI.S1, LAN_PI.S2, R33.1, R34.1, R35.2, RPI.14, RPI.20, RPI.25, RPI.30, RPI.34, RPI.39, RPI.6, RPI.9, SV6.1; no longer C2.2, IC1B.I0, IC1B.I1, IC1C.I0, IC1C.I1, IC1D.I0, IC1D.I1, IC1P.GND, IC2CE.E, IC3CE.E, NS2-4.1, R6.1, SV1.14, SV1.20, SV1.25, SV1.6, SV1.9, U3A.S
- net GNDA: now also C2.2, C21.2, C24.2, C3.2, C34.2, C37.2, C38.2, C5.2, IC1.GND2, IC10.GND2@1, IC10.GND2@2, IC11.GND2@1, IC11.GND2@2, IC15.GND, IC16A.S, IC2.GND1@1, IC2.GND1@2, IC3.GND1@1, IC3.GND1@2, IC9.GND2@1, IC9.GND2@2, R6.1, TP_IGND.MP, TP_IGND1.MP; no longer IGND.MP, Q1.S, Q2.S
- net MISO: now also RPI.21; no longer SV1.21
- net MOSI: now also RPI.19; no longer SV1.19
- net N$11: now also IC10.INC, IC2.OUTC, R22.1; no longer IC2LED.A, R2.2
- net N$12: now also IC3.INA, IC9.OUTA, R25.1; no longer IC3LED.A, R3.2
- net N$14: now also IC10.OUTC, IC2.INC, R4.1; no longer IC3LED.K, Q2.D
- net N$2: now also IC10.OUTA, IC2.INA, R2.1; no longer IC2LED.K, Q1.D
- net N$3: now also IC16A.G; no longer U3A.G
- net N$4: now also IC16B.G; no longer U3B.G
- net N$8: now also IC16A.D; no longer U3A.D
- net RXD: now also IC14.20_TXD/SPI_MISO, RPI.10; no longer NS1-2.1, SV1.10
- net SCLK: now also RPI.23; no longer SV1.23
- net TXD: now also IC14.21_RXD/SPI_MOSI, RPI.8; no longer NS1-1.1, SV1.8
- net V-: now also USB_TGT.4; no longer USB_TARGET.4
- net VBUS: now also C4.1, L1.1; no longer R9.2, U3B.S
- net VCC: now also C37.1, IC15.EN, IC15.VIN, IC16B.S, R9.2; no longer R2.1, R3.1, USB_TARGET.1, V.1
Other:
- note added: "3.3V Target Power (Isolated side)"
- note added: "Close to PI"
- note added: "Close to inverters"
- note added: "Close to isolators, one on each side"
- note added: "Control Block Isolation"
- note added: "Isolated EEPROM"
- note added: "Isolation Block 1"
- note added: "Isolation Block 2"
- note added: "PoE In (from Switch)"
- note added: "PoE Module"
- note added: "RJ45 Out (to Pi)"
- note added: "RPI 40 Pin Connector"
- note added: "Target Connectors"
- note added: "U-BLOX GPS"
- note added: "Weak Pull-Up to ensure as little current as possible may be leaked here."
- note removed: "Edge Detector (Use C1 and R1 for timing)"
- note removed: "Navspark Connector"
- note removed: "RPI 26 Pin Connector"
- note removed: "Remaining Pins for 40 Pin Variants"
- note removed: "Target Connector"
